File: eagle/fullcircuit4layer1.1b.sch (EAGLE design)
At the start: 117 parts, among them IC1 MCP1703CB, U1 MIC5219 5V, U3 MIC5219 3.3V, X1 TXC_7A

Commit message: updated schematic with missing values corrected PCB layout
Parts:
- added R14: 1K, SparkFun-Passives:RESISTOR0603-RES
- C22: value (none) -> NF
- C26, C27: value 4pF -> 3.9pF
- Q1: value (none) -> MMBT5088
- Q2: value (none) -> MMBT4403
- R2, R3, R8: value (none) -> 100R
- R4: value (none) -> 220R
- U$1: value STM32F302XX -> STM32F302CBT6
- U$7: value AFT0SMS003N -> AFT05MS003NT1
Connections:
- new net N$109: C13.1, R14.1
- net ANT: now also R14.2; no longer C13.1
- net GND: now also U$6.GND@7
